File: pcb/tairakb.kicad_sch (KiCad schematic)
At the start: 79 parts, among them SW1 SW_Push, SW10 SW_Push, SW11 SW_Push, SW12 SW_Push, SW13 SW_Push, SW14 SW_Push, SW15 SW_Push, SW16 SW_Push, SW17 SW_Push, SW18 SW_Push, SW19 SW_Push, SW2 SW_Push, SW20 SW_Push, SW20-1 SW_Push, SW21 SW_Push, SW22 SW_Push, SW23 SW_Push, SW24 SW_Push, SW25 SW_Push, SW26 SW_Push, SW27 SW_Push, SW28 SW_Push, SW29 SW_Push, SW3 SW_Push, SW30 SW_Push, SW31 SW_Push, SW32 SW_Push, SW33 SW_Push, SW4 SW_Push, SW5 SW_Push, SW6 SW_Push, SW7 SW_Push, SW8 SW_Push, SW9 SW_Push, U3 nice!nano

Commit message: remove outermost two thumb keys (SW32, SW33)
Shrinks the thumb cluster from 5 to 3 keys (SW25, SW30, SW31 remain).
Deletes the footprints, schematic symbols, orphan D32/D33-Pad2 traces,
and the dangling /col6 segments/vias in the cut region; trims Edge.Cuts
on the PCB and both plates to wrap only the remaining keys (H8 stays
enclosed). DRC stays at the pre-existing 4-violation baseline; ERC
clean.

Co-Authored-By: Claude Opus 4.7 <noreply@anthropic.com>
Parts:
- removed D32, D33: D, tairakb:D3_SMD, symbol Device:D
- removed SW32, SW33: SW_Push, tairakb:Choc_Hotswap, symbol Switch:SW_Push

Commit message: 1.5U bottom thumb + thumb cluster reflow (Pass A)
SW30 enlarged to 1.5U using a new Choc_Hotswap_1.5U footprint (no
stabilizers); the keycap's bottom edges are anchored, so the switch
center shifts up-and-right to (194.515, 133.274). SW31 rotated from
-30° to 180° and placed beside SW29 in the next main-grid column at
(201.295, 106.594). U3 moved up to (204.445, 61.112) so its top edge
aligns with SW26; PCB and both plate Edge.Cuts extended in the
controller area to give U3 the needed vertical room. RSW1, BSW1, BT1
shifted up 15mm to clear the new SW31 and U3 envelopes. Schematic
SW30 footprint property updated to match.

Pass A only: trace endpoints near moved pads have been nudged or, for
SW31's deleted pad stubs, removed. Broader re-routing in KiCad GUI is
pending and will land in a follow-up commit; DRC currently reports
~495 violations in the affected region.

Co-Authored-By: Claude Opus 4.7 <noreply@anthropic.com>
Parts:
- SW30: footprint tairakb:Choc_Hotswap -> tairakb:Choc_Hotswap_1.5U
Changed lines of the file:
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@@
 			)
 		)
-		(property "Footprint" "tairakb:Choc_Hotswap"
+		(property "Footprint" "tairakb:Choc_Hotswap_1.5U"
 			(at 250.19 76.2 0)
 			(hide yes)
